File: PCB/Hackpad PCB.kicad_pcb (KiCad board)
At the start: 2 copper layers, 112 x 75 mm, 12 parts, among them SW1 SW_Push, SW2 SW_Push, SW3 SW_Push, SW4 SW_Push, SW5 SW_Push, SW6 SW_Push, SW7 SW_Push, SW8 SW_Push, SW9 SW_Push, U1 XIAO-RP2040-DIP

Commit message: Add files via upload
Parts:
- moved D2 20.0 mm to (95.5, 90.5), turned to -90 degrees
- moved D1 15.1 mm to (101.5, 90.5), turned to -90 degrees
- moved U1 11.4 mm to (98.4, 74.3)
Routing:
- net +5V: track 154.8 -> 38.5 mm
- net Net-(U1-GPIO7/SCL): track 68.4 -> 159.0 mm
- net Net-(U1-GPIO6/SDA): track 62.7 -> 142.5 mm
- net Net-(U1-GPIO0/TX): track 163.8 -> 92.2 mm
- net Net-(D1-DIN): track 62.6 -> 17.7 mm
- net Net-(U1-GPIO29/ADC3/A3): track 72.9 -> 54.1 mm
- net Net-(U1-GPIO26/ADC0/A0): track 49.7 -> 34.1 mm
- net Net-(U1-GPIO27/ADC1/A1): track 50.9 -> 42.1 mm
- net GND: track 219.1 -> 210.6 mm
- net Net-(D1-DOUT): track 14.5 -> 9.20 mm
- net Net-(U1-GPIO2/SCK): track 89.6 -> 86.4 mm
- net Net-(U1-GPIO28/ADC2/A2): track 68.2 -> 70.5 mm
- net Net-(U1-GPIO1/RX): track 80.6 -> 82.1 mm
Other:
- board size 112 x 75 mm -> 89 x 69 mm
